Commit message: lots of glider things

File: ros_pat/urdf/fox.urdf.xacro (robot description, xacro)
@@ -3,5 +3,6 @@
   <xacro:property name="robot_name" value="fox" />
   <xacro:property name="high_definition_fuselage_visual" value="true" />
-  <xacro:property name="high_definition_wing_visual" value="false" />
+  <xacro:property name="fuselage_mesh" value="package://ros_pat/media/glider.dae" />
+  <xacro:property name="high_definition_wing_visual" value="true" />
   <xacro:property name="high_definition_ele_visual" value="true" />
   <!-- Fuselage -->

File: ros_pat/urdf/glider.urdf.xacro (robot description, xacro)
@@ -9,5 +9,5 @@
 	<origin xyz="0 0 0" rpy="0 0 0"/>
         <geometry>
-	  <mesh scale="1. 1. 1." filename="package://ros_pat/media/glider.dae"/>
+	  <mesh scale="1. 1. 1." filename="${fuselage_mesh}"/>
         </geometry>
       </xacro:if>

File: ros_pat/urdf/vtail_glider.urdf.xacro (robot description, xacro)
@@ -19,8 +19,4 @@
       </xacro:unless>
     </visual>
-    <xacro:inertial_cuboid_with_pose
-	mass="${fuselage_m}" x_length="${fuselage_l}" y_length="${fuselage_w}" z_length="${fuselage_h}">
-      <origin xyz="0 0 0" rpy="0 0 0"/>
-    </xacro:inertial_cuboid_with_pose>
   </link>
   <joint name="fuselage_link_joint" type="fixed">
